Commit message: chassis link merged into base_link

File: src/erp42_racing_description/urdf/erp42_racing_model.xacro (robot description, xacro)
@@ -27,7 +27,5 @@
         <link name="base_footprint"/>
         <!-- Base link -->
-        <link name="base_link"/>
-        <!-- Chassis -->
-        <link name="chassis">
+        <link name="base_link">
             <!-- Inertia -->
             <inertial>
@@ -104,10 +102,4 @@
             <child link="base_link" />
         </joint>
-        <!-- base_link to chassis -->
-        <joint name="chassis_joint" type="fixed">
-            <origin xyz="0 0 0" rpy="0 0 0" />
-            <parent link="base_link" />
-            <child link="chassis" />
-        </joint>
         <!-- base_link to front_left_steering_hub -->
         <joint name="front_left_steering_hub_joint" type="revolute">
