Commit message: Odometry data publication flag added

File: src/erp42_racing_gazebo/urdf/erp42_racing_gazebo.xacro (robot description, xacro)
@@ -2,8 +2,6 @@
 <robot xmlns:xacro="http://ros.org/wiki/xacro" name="erp42_racing">
     <!-- Include files -->
-    <xacro:include filename="$(find erp42_racing_description)/urdf/erp42_racing_model.xacro"/>
     <xacro:include filename="$(find erp42_racing_gazebo)/urdf/erp42_racing_gazebo_control.xacro"/>
     <!-- ERP42 Racing model description and gazebo control settings -->
-    <xacro:erp42_racing_model/>
-    <xacro:erp42_racing_gazebo_control/>
+    <xacro:erp42_racing_gazebo_control publish_odometry = "true" />
 </robot>

File: src/erp42_racing_gazebo/urdf/erp42_racing_gazebo_control.xacro (robot description, xacro)
@@ -1,5 +1,8 @@
 <?xml version="1.0"?>
 <robot xmlns:xacro="http://ros.org/wiki/xacro">
-    <xacro:macro name="erp42_racing_gazebo_control" params="">
+    <xacro:macro name="erp42_racing_gazebo_control" params="publish_odometry">
+        <!-- ERP42 Racing model -->
+        <xacro:include filename="$(find erp42_racing_description)/urdf/erp42_racing_model.xacro"/>
+        <xacro:erp42_racing_model/>
         <!-- Friction coefficients -->
         <gazebo reference="front_left_wheel">
@@ -65,6 +68,6 @@
                 <linear_velocity_i_range>0 0</linear_velocity_i_range>
                 <!-- Odometry parameters -->
-                <publish_odom>true</publish_odom>
-                <publish_odom_tf>true</publish_odom_tf>
+                <publish_odom>${publish_odometry}</publish_odom>
+                <publish_odom_tf>${publish_odometry}</publish_odom_tf>
                 <odometry_frame>odom</odometry_frame>
                 <robot_base_frame>base_footprint</robot_base_frame>
