Commit message: Vehicle parameter edited

File: src/erp42_racing_gazebo_sim/urdf/erp42_racing_description.xacro (robot description, xacro)
@@ -51,5 +51,8 @@
         />
         <gazebo>
-            <plugin name="gz::sim::systems::JointStatePublisher" filename="gz-sim-joint-state-publisher-system">
+            <plugin
+                name="gz::sim::systems::JointStatePublisher"
+                filename="gz-sim-joint-state-publisher-system"
+            >
                 <!-- Update rate -->
                 <update_rate>100.0</update_rate>
@@ -62,11 +65,14 @@
                 <joint_name>rear_right_wheel_joint</joint_name>
             </plugin>
-            <plugin name="gz::sim::systems::ERP42RacingControl" filename="liberp42_racing_control.so">
-                <left_steer_joint>front_left_wheel_steer_joint</left_steer_joint>
-                <right_steer_joint>front_right_wheel_steer_joint</right_steer_joint>
-                <front_left_joint>front_left_wheel_joint</front_left_joint>
-                <front_right_joint>front_right_wheel_joint</front_right_joint>
-                <rear_left_joint>rear_left_wheel_joint</rear_left_joint>
-                <rear_right_joint>rear_right_wheel_joint</rear_right_joint>
+            <plugin
+                name="gz::sim::systems::ERP42RacingGazeboControl"
+                filename="liberp42_racing_gazebo_control.so"
+            >
+                <left_steering_joint>front_left_wheel_steer_joint</left_steering_joint>
+                <right_steering_joint>front_right_wheel_steer_joint</right_steering_joint>
+                <front_left_wheel_joint>front_left_wheel_joint</front_left_wheel_joint>
+                <front_right_wheel_joint>front_right_wheel_joint</front_right_wheel_joint>
+                <rear_left_wheel_joint>rear_left_wheel_joint</rear_left_wheel_joint>
+                <rear_right_wheel_joint>rear_right_wheel_joint</rear_right_wheel_joint>
                 <wheel_base>${wheelbase}</wheel_base>
                 <kingpin_width>${front_tread}</kingpin_width>
@@ -75,9 +81,9 @@
                 <front_wheel_radius>${front_wheel_radius}</front_wheel_radius>
                 <rear_wheel_radius>${rear_wheel_radius}</rear_wheel_radius>
-                <steer_limit>${radians(20)}</steer_limit>
-                <steer_p_gain>10.0</steer_p_gain>
+                <steering_p_gain>10.0</steering_p_gain>
+                <steering_limit>${radians(20)}</steering_limit>
                 <velocity_limit>5.5</velocity_limit>
-                <acceleration_limit>2.0</acceleration_limit>
-                <brake_deceleration>15.0</brake_deceleration>
+                <acceleration_limit>2.5</acceleration_limit>
+                <brake_deceleration>10.0</brake_deceleration>
                 <publish_odometry>${publish_odometry}</publish_odometry>
                 <odometry_frequency>100.0</odometry_frequency>

File: src/erp42_racing_gazebo_sim/urdf/erp42_racing_front_wheel.xacro (robot description, xacro)
@@ -84,11 +84,11 @@
             <axis xyz = "0 0 1"/>
             <!-- Dynamics -->
-            <dynamics friction = "10.0" damping = "1.0"/>
+            <dynamics friction = "0.1" damping = "0.1"/>
             <!-- Limits -->
             <limit
-                lower    = "${-1.2 * radians(25)}"
-                upper    = "${ 1.2 * radians(25)}"
-                effort   = "1000"
-                velocity = "1.0"
+                lower    = "${-1.2 * radians(20)}"
+                upper    = "${ 1.2 * radians(20)}"
+                velocity = "${ 2.0 * radians(20)}"
+                effort   = "1000000.0"
             />
         </joint>
@@ -103,10 +103,10 @@
             <axis xyz = "0 1 0"/>
             <!-- Limits -->
-            <limit effort = "10000.0" velocity = "${7.0 / radius}"/>
+            <limit effort = "1000000.0" velocity = "${10.0 / radius}"/>
         </joint>
         <!-- Friction settings -->
         <gazebo reference="${wheel_link}">
-            <mu1>0.9</mu1>
-            <mu2>0.9</mu2>
+            <mu1>0.75</mu1>
+            <mu2>0.75</mu2>
         </gazebo>
     </xacro:macro>

File: src/erp42_racing_gazebo_sim/urdf/erp42_racing_rear_wheel.xacro (robot description, xacro)
@@ -55,5 +55,5 @@
             <axis xyz = "0 1 0"/>
             <!-- Limits -->
-            <limit effort = "10000.0" velocity = "${7.0 / radius}"/>
+            <limit effort = "1000000.0" velocity = "${10.0 / radius}"/>
         </joint>
         <!-- Friction settings -->

Commit message: Vehicle parameter edited

File: src/erp42_racing_gazebo_sim/urdf/erp42_racing_description.xacro (robot description, xacro)
@@ -81,5 +81,5 @@
                 <front_wheel_radius>${front_wheel_radius}</front_wheel_radius>
                 <rear_wheel_radius>${rear_wheel_radius}</rear_wheel_radius>
-                <steering_p_gain>10.0</steering_p_gain>
+                <steering_p_gain>100.0</steering_p_gain>
                 <steering_limit>${radians(20)}</steering_limit>
                 <velocity_limit>5.5</velocity_limit>

File: src/erp42_racing_gazebo_sim/urdf/erp42_racing_front_wheel.xacro (robot description, xacro)
@@ -13,5 +13,5 @@
         <xacro:property name  = "izz" value = "${1/2  * mass * radius * radius}"/>
         <!-- Steer properties -->
-        <xacro:property name = "dummy_mass"   value = "5"  />
+        <xacro:property name = "dummy_mass"   value = "1"  />
         <xacro:property name = "dummy_radius" value = "0.1"/>
         <xacro:property name = "dummy_ixx" value = "${3/5 * dummy_mass * dummy_radius * dummy_radius}"/>
@@ -89,5 +89,5 @@
                 lower    = "${-1.2 * radians(20)}"
                 upper    = "${ 1.2 * radians(20)}"
-                velocity = "${ 2.0 * radians(20)}"
+                velocity = "${ 4.0 * radians(20)}"
                 effort   = "1000000.0"
             />
@@ -103,10 +103,10 @@
             <axis xyz = "0 1 0"/>
             <!-- Limits -->
-            <limit effort = "1000000.0" velocity = "${10.0 / radius}"/>
+            <limit effort = "360.0" velocity = "${5.5 / radius}"/>
         </joint>
         <!-- Friction settings -->
         <gazebo reference="${wheel_link}">
-            <mu1>0.75</mu1>
-            <mu2>0.75</mu2>
+            <mu1>0.9</mu1>
+            <mu2>0.9</mu2>
         </gazebo>
     </xacro:macro>

File: src/erp42_racing_gazebo_sim/urdf/erp42_racing_rear_wheel.xacro (robot description, xacro)
@@ -55,5 +55,5 @@
             <axis xyz = "0 1 0"/>
             <!-- Limits -->
-            <limit effort = "1000000.0" velocity = "${10.0 / radius}"/>
+            <limit effort = "360.0" velocity = "${5.5 / radius}"/>
         </joint>
         <!-- Friction settings -->
