Commit message: Modify origin z-coordinate in front wheel xacro
Adjusted the origin's z-coordinate for the front wheel.

File: src/erp42_racing_gazebo_sim/urdf/erp42_racing_front_wheel.xacro (robot description, xacro)
@@ -80,5 +80,5 @@
             <child  link = "${wheel_link}_steer"/>
             <!-- Origin -->
-            <origin xyz = "${wheelbase/2} ${reflection * tread/2} 0" rpy = "0 0 0"/>
+            <origin xyz = "${wheelbase/2} ${reflection * tread/2} -0.01" rpy = "0 0 0"/>
             <!-- Rotation axis -->
             <axis xyz = "0 0 1"/>
